File: pcb_ctrl_esp5v/pcb_ctrl_esp5v.sch (KiCad schematic (older format))
At the start: 7 parts, among them J1 USB_B_Micro, J2 Barrel_Jack, SW1 SW_SPST, SW2 SW_SPST, U1 ESP32-WROOM, U2 LM1117-ADJ, U3 FT232RL

Commit message: working on ctrl pcb
Parts:
- added C1, C10, C3, C4, C6, C7, C8, C9: 100n, Capacitor_SMD:C_0805_2012Metric_Pad1.15x1.40mm_HandSolder, symbol Device:C
- added C2: 10u, Capacitor_SMD:C_0805_2012Metric_Pad1.15x1.40mm_HandSolder, symbol Device:C
- added C5: 4.7u, Capacitor_SMD:C_0805_2012Metric_Pad1.15x1.40mm_HandSolder, symbol Device:C
- added J3: Conn_02x10_Odd_Even, Connector_PinSocket_2.54mm:PinSocket_2x10_P2.54mm_Vertical, symbol Connector_Generic:Conn_02x10_Odd_Even
- added J4: Conn_01x03, Connector_PinSocket_2.54mm:PinSocket_1x03_P2.54mm_Vertical, symbol Connector_Generic:Conn_01x03
- added Q1, Q2: S8050, Package_TO_SOT_THT:TO-92_Inline, symbol Transistor_BJT:S8050
- added R1, R2, R4: 10k, Resistor_SMD:R_0805_2012Metric_Pad1.15x1.40mm_HandSolder, symbol Device:R
- added R3: 4.7k, Resistor_SMD:R_0805_2012Metric_Pad1.15x1.40mm_HandSolder, symbol Device:R
- added R5: 121, Resistor_SMD:R_0805_2012Metric_Pad1.15x1.40mm_HandSolder, symbol Device:R
- added R6: 200, Resistor_SMD:R_0805_2012Metric_Pad1.15x1.40mm_HandSolder, symbol Device:R
- added U4: 74HC00, Package_SO:SOIC-14_3.9x8.7mm_P1.27mm, symbol 74xx:74HC00
Connections:
- net labels added: +3.3V, +5V, DOUT, DOUT_33, DTR, EN, GND, IO0, IO12, IO13, IO14, IO25, IO26, IO27, IO32, IO33, IO34, IO35, RTS, RXD0, SENSOR_VN, SENSOR_VP, TXD0
- wire segments 0 -> 177
- no-connect marks 0 -> 23
Other:
- note added: "5 V Input + 3.3 V Reg"
- note added: "Connectors"
- note added: "ESP32 Controller"
- note added: "Level shift"
- note added: "Setup switches"
- note added: "USB to UART"

Commit message: pretty much ready to order now, checks required
Parts:
- removed Q1, Q2: S8050, Package_TO_SOT_THT:TO-92_Inline, symbol Transistor_BJT:S8050
- added Q1, Q2: S8050 SOT-23, Package_TO_SOT_SMD:SOT-23_Handsoldering, symbol Device:Q_NPN_BEC
Changed lines of the file:
@@
 Wire Wire Line
 	4050 4650 4550 4650
-$Comp
-L Transistor_BJT:S8050 Q1
-U 1 1 5C62FB64
-P 1850 6500
-F 0 "Q1" H 2041 6546 50  0000 L CNN
-F 1 "S8050" H 2041 6455 50  0000 L CNN
-F 2 "Package_TO_SOT_THT:TO-92_Inline" H 2050 6425 50  0001 L CIN
-F 3 "http://www.unisonic.com.tw/datasheet/S8050.pdf" H 1850 6500 50  0001 L CNN
-	1    1850 6500
-	1    0    0    -1
-$EndComp
-$Comp
-L Transistor_BJT:S8050 Q2
-U 1 1 5C62FD03
-P 1850 7150
-F 0 "Q2" H 2041 7104 50  0000 L CNN
-F 1 "S8050" H 2041 7195 50  0000 L CNN
-F 2 "Package_TO_SOT_THT:TO-92_Inline" H 2050 7075 50  0001 L CIN
-F 3 "http://www.unisonic.com.tw/datasheet/S8050.pdf" H 1850 7150 50  0001 L CNN
-	1    1850 7150
-	1    0    0    1
-$EndComp
 Text Label 950  7150 2    50   ~ 0
 RTS
@@
 Text Notes 5200 3400 0    118  ~ 0
 Level shift
+$Comp
+L Device:Q_NPN_BEC Q1
+U 1 1 5C898189
+P 1850 6500
+F 0 "Q1" H 2041 6546 50  0000 L CNN
+F 1 "S8050 SOT-23" H 2041 6455 50  0000 L CNN
+F 2 "Package_TO_SOT_SMD:SOT-23_Handsoldering" H 2050 6600 50  0001 C CNN
+F 3 "~" H 1850 6500 50  0001 C CNN
+	1    1850 6500
+	1    0    0    -1
+$EndComp
+$Comp
+L Device:Q_NPN_BEC Q2
+U 1 1 5C8A0E4E
+P 1850 7150
+F 0 "Q2" H 2041 7104 50  0000 L CNN
+F 1 "S8050 SOT-23" H 2041 7195 50  0000 L CNN
+F 2 "Package_TO_SOT_SMD:SOT-23_Handsoldering" H 2050 7250 50  0001 C CNN
+F 3 "~" H 1850 7150 50  0001 C CNN
+	1    1850 7150
+	1    0    0    1
+$EndComp
 $EndSCHEMATC

Commit message: ERC clean
Connections:
- wire segments 177 -> 179
- no-connect marks 23 -> 30
Changed lines of the file:
@@
-	1    0    0    -1
-$EndComp
-$Comp
-L power:+5V #PWR0101
-U 1 1 5C60884D
-P 2800 1200
-F 0 "#PWR0101" H 2800 1050 50  0001 C CNN
-F 1 "+5V" H 2815 1373 50  0000 C CNN
-F 2 "" H 2800 1200 50  0001 C CNN
-F 3 "" H 2800 1200 50  0001 C CNN
-	1    2800 1200
 	1    0    0    -1
 $EndComp
@@
 Wire Wire Line
 	10000 1800 10200 1800
-Wire Wire Line
-	10000 1650 10000 1700
-Wire Wire Line
-	10000 1700 10200 1700
 Wire Wire Line
 	10000 1950 10000 1900
@@
 	4550 2000 4550 1850
 Wire Wire Line
-	1700 1350 2800 1350
+	1700 1350 2050 1350
 Wire Wire Line
 	2800 1200 2800 1350
@@
 L power:+5V #PWR0124
 U 1 1 5C6AB690
-P 9150 1250
-F 0 "#PWR0124" H 9150 1100 50  0001 C CNN
-F 1 "+5V" H 9165 1423 50  0000 C CNN
-F 2 "" H 9150 1250 50  0001 C CNN
-F 3 "" H 9150 1250 50  0001 C CNN
-	1    9150 1250
-	1    0    0    -1
-$EndComp
-Wire Wire Line
-	8850 1450 9150 1450
-Wire Wire Line
-	9150 1450 9150 1250
+P 9200 1250
+F 0 "#PWR0124" H 9200 1100 50  0001 C CNN
+F 1 "+5V" H 9215 1423 50  0000 C CNN
+F 2 "" H 9200 1250 50  0001 C CNN
+F 3 "" H 9200 1250 50  0001 C CNN
+	1    9200 1250
+	1    0    0    -1
+$EndComp
 Wire Wire Line
 	8350 1450 8050 1450
@@
 	1    0    0    1
 $EndComp
+NoConn ~ 1400 4950
+NoConn ~ 1000 5150
+NoConn ~ 4050 5450
+NoConn ~ 4050 5550
+NoConn ~ 4050 5650
+NoConn ~ 4050 5750
+NoConn ~ 4050 5850
+Wire Wire Line
+	9200 1450 8850 1450
+Wire Wire Line
+	9200 1250 9200 1450
+Wire Wire Line
+	10000 1650 10000 1700
+Wire Wire Line
+	10000 1700 10200 1700
+$Comp
+L power:+5V #PWR0101
+U 1 1 5C692B51
+P 2800 1200
+F 0 "#PWR0101" H 2800 1050 50  0001 C CNN
+F 1 "+5V" H 2815 1373 50  0000 C CNN
+F 2 "" H 2800 1200 50  0001 C CNN
+F 3 "" H 2800 1200 50  0001 C CNN
+	1    2800 1200
+	1    0    0    -1
+$EndComp
+$Comp
+L power:PWR_FLAG #FLG0101
+U 1 1 5C692CA3
+P 2050 1250
+F 0 "#FLG0101" H 2050 1325 50  0001 C CNN
+F 1 "PWR_FLAG" H 2050 1424 50  0000 C CNN
+F 2 "" H 2050 1250 50  0001 C CNN
+F 3 "~" H 2050 1250 50  0001 C CNN
+	1    2050 1250
+	1    0    0    -1
+$EndComp
+Wire Wire Line
+	2050 1250 2050 1350
+Connection ~ 2050 1350
+Wire Wire Line
+	2050 1350 2800 1350
 $EndSCHEMATC
