File: pcb_ctrl_esp5v/pcb_ctrl_esp5v.kicad_pcb (KiCad board)
At the start: 2 copper layers, 86.4 x 75 mm, 34 parts, among them J1 USB_B_Micro, J2 Barrel_Jack, J3 Conn_02x10_Odd_Even, J4 Conn_01x03, Q1 S8050, Q2 S8050, SW1 SW_SPST, SW2 SW_SPST, U1 ESP32-WROOM, U2 LM1117-ADJ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

Commit message: pretty much ready to order now, checks required
Parts:
- Q1, Q2: value S8050 -> S8050 SOT-23; footprint Package_TO_SOT_THT:TO-92_Inline -> Package_TO_SOT_SMD:SOT-23_Handsoldering
- moved R1 101.2 mm to (108.1, 110.7)
- moved R2 98.9 mm to (108.0, 116.0)
- moved C5 97.5 mm to (109.6, 98.8), turned to 270 degrees
- moved C8 93.7 mm to (109.6, 94.5), turned to 90 degrees
- moved R3 93.2 mm to (113.8, 85.6), turned to 90 degrees
- moved C1 93.1 mm to (113.9, 90.1), turned to 90 degrees
- moved R4 89.0 mm to (118.0, 85.6), turned to 90 degrees
- moved C7 88.0 mm to (120.5, 77.0), turned to 90 degrees
- moved C4 82.1 mm to (113.9, 94.4), turned to 90 degrees
- moved C3 82.1 mm to (113.9, 98.7), turned to 270 degrees
- moved R6 71.0 mm to (133.0, 81.0), turned to 90 degrees
- moved C6 70.8 mm to (133.0, 86.0), turned to 270 degrees
- moved R5 63.9 mm to (136.5, 81.0), turned to 90 degrees
- moved C9 63.2 mm to (136.3, 93.6)
- moved C2 57.3 mm to (136.5, 86.0), turned to 270 degrees
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Connections:
- Q1 pad 1: /RTS -> Net-(Q1-Pad1)
- Q1 pad 2: Net-(Q1-Pad2) -> /RTS
- Q2 pad 1: /DTR -> Net-(Q2-Pad1)
- Q2 pad 2: Net-(Q2-Pad2) -> /DTR
- R1 pad 1: Net-(Q1-Pad2) -> Net-(Q1-Pad1)
- R2 pad 1: Net-(Q2-Pad2) -> Net-(Q2-Pad1)
Routing:
- net /EN: track 0.00 -> 160.8 mm, vias 0 -> 2
- net GND: track 0.00 -> 141.8 mm, vias 0 -> 20
- net /IO0: track 0.00 -> 104.4 mm, vias 0 -> 2
- net +5V: track 0.00 -> 98.4 mm, vias 0 -> 3
- net /RXD0: track 0.00 -> 86.9 mm, vias 0 -> 4
- net /TXD0: track 0.00 -> 74.6 mm, vias 0 -> 3
- net /IO13: track 0.00 -> 55.7 mm, vias 0 -> 3
- net +3V3: track 0.00 -> 51.4 mm, vias 0 -> 4
- net /DTR: track 0.00 -> 48.5 mm, vias 0 -> 2
- net /IO14: track 0.00 -> 47.4 mm, vias 0 -> 3
- net /IO25: track 0.00 -> 45.9 mm, vias 0 -> 2
- net /SENSOR_VN: track 0.00 -> 45.6 mm
- net /IO26: track 0.00 -> 44.8 mm, vias 0 -> 1
- net /IO12: track 0.00 -> 43.3 mm
- net /IO33: track 0.00 -> 43.1 mm, vias 0 -> 1
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- added copper zone on B.Cu, net +3V3
- added copper zone on B.Cu, net +5V
- added copper zone on B.Cu, net GND
- added copper zone on F.Cu, net GND
Other:
- net class Default: trace_width 0.25 -> 0.3
- rule via_min_drill: 0.3 -> 0.4
- rule via_min_size: 0.4 -> 0.8

Commit message: DRC clean - ordering this now
Parts:
- added REF**: TestPoint_THTPad_2.5x2.5mm_Drill1.2mm, TestPoint:TestPoint_THTPad_2.5x2.5mm_Drill1.2mm, F.Cu at (109.0, 105.3)
Routing:
- net /EN: track 160.8 -> 145.1 mm, vias 2 -> 5
- net (no net): track 8.85 -> 0.00 mm, vias 2 -> 0
- net /DTR: track 48.5 -> 43.7 mm
- net GND: track 141.8 -> 137.7 mm, vias 20 -> 26
- net +3V3: track 51.4 -> 54.6 mm
- net /IO14: track 47.4 -> 45.3 mm
- net +5V: track 98.4 -> 96.9 mm
- net Net-(C1-Pad1): track 16.8 -> 15.7 mm
- net /RXD0: track 86.9 -> 85.9 mm
- net /DOUT_33: track 41.9 -> 41.1 mm
- net /RTS: track 34.2 -> 34.8 mm
Other:
- board text added: "5V DC center+"
- board text added: "GND"
- board text added: "Tobias Kaiser netlantern pcb_ctrl_esp5v Feb 12 2019"
